File: current_sense_2026.kicad_sch (KiCad schematic)
At the start: 0 parts

Commit message: Push Test
Parts:
- added C1: C, Package_QFP:TQFP-44_10x10mm_P0.8mm, symbol Device:C
Changed lines of the file:
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@@
 	(generator_version "10.0")
 	(paper "A4")
+	(symbol
+		(lib_id "Device:C")
+		(at 138.43 91.44 0)
+		(unit 1)
+		(body_style 1)
+		(exclude_from_sim no)
+		(in_bom yes)
+		(on_board yes)
+		(in_pos_files yes)
+		(dnp no)
+		(fields_autoplaced yes)
+		(property "Reference" "C1"
+			(at 142.24 90.1699 0)
+			(show_name no)
+			(do_not_autoplace no)
+			(effects
+				(font
+					(size 1.27 1.27)
+				)
+				(justify left)
+			)
+		)
+		(property "Value" "C"
+			(at 142.24 92.7099 0)
+			(show_name no)
+			(do_not_autoplace no)
+			(effects
+				(font
+					(size 1.27 1.27)
+				)
+				(justify left)
+			)
+		)
+		(property "Footprint" "Package_QFP:TQFP-44_10x10mm_P0.8mm"
+			(at 139.3952 95.25 0)
+			(hide yes)
+			(show_name no)
+			(do_not_autoplace no)
+			(effects
+				(font
+					(size 1.27 1.27)
+				)
+			)
+		)
+		(property "Datasheet" ""
+			(at 138.43 91.44 0)
+			(hide yes)
+			(show_name no)
+			(do_not_autoplace no)
+			(effects
+				(font
+					(size 1.27 1.27)
+				)
+			)
+		)
+		(property "Description" "Unpolarized capacitor"
+			(at 138.43 91.44 0)
+			(hide yes)
+			(show_name no)
+			(do_not_autoplace no)
+			(effects
+				(font
+					(size 1.27 1.27)
+				)
+			)
+		)
+		(pin "1"
+		)
+		(pin "2"
+		)
+		(instances
+			(project "current_sense_2026"
+				(path "/36598e4c-76b2-4a5e-9408-b8c253e2f1ff"
+					(reference "C1")
+					(unit 1)
+				)
+			)
+		)
+	)
 	(sheet_instances
 		(path "/"

Commit message: Battery Update 10/24/2026 11:50 a.m.
Outline for the schematic
Parts:
- added C2, C3, C4: 0.1u, Capacitor_SMD:C_1206_3216Metric, symbol Device:C
- added C5: 1u, Capacitor_SMD:C_1206_3216Metric, symbol Device:C
- added J1: Conn_01x04_Socket, Connector_JST:JST_XH_B4B-XH-A_1x04_P2.50mm_Vertical, symbol Connector:Conn_01x04_Socket
- added J2: Conn_01x04_Pin, Connector_JST:JST_XH_B4B-XH-A_1x04_P2.50mm_Vertical, symbol Connector:Conn_01x04_Pin
- added U1: NAU7802KGI, Package_DIP:DIP-16_W7.62mm, symbol 2026-2027_Battery_Symbols:NAU7802KGI
- added U2: (no value), Library:DFR1193, symbol 2026-2027_Battery_Symbols:DFR1193
- C1: value C -> 0.1u; footprint Package_QFP:TQFP-44_10x10mm_P0.8mm -> Capacitor_SMD:C_1206_3216Metric
Connections:
- net +5V: now reaches C1.1
- net +5V: now also C3.2, J1.1 (Pin_1), J2.4 (Pin_4), U1.1 (REFP), U1.15 (DVDD), U2.1 (VCC1), U2.9 (VCC2)
- net GND: now reaches C1.2
- net GND: now also C2.2, C3.1, C4.2, C5.2, J1.2 (Pin_2), J2.3 (Pin_3), U1.4 (VIN2N), U1.7 (REFN), U1.8 (AVSS), U1.9 (DVSS), U2.2 (GND1), U2.8 (GND2)
- new net: C2.1, C5.1, U1.16 (AVDD/LDO)
- new net: C4.1, U1.6 (VBG)
- new net SCL_In: U1.13 (SCLK), U2.3 (SCL_IN)
- new net SCL_Out: J2.1 (Pin_1), U2.7 (SCL_OUT)
- new net SDA_In: U1.14 (SDIO), U2.4 (SDA_IN)
- new net SDA_Out: J2.2 (Pin_2), U2.6 (SDA_OUT)
- new net SENSE1_OUT: J1.4 (Pin_4), U1.5 (VIN2P)
- no-connect marks 0 -> 8
