File: Linear Actuator/Linear Actuator.kicad_sch (KiCad schematic)
At the start: 0 parts

Commit message: Fixed Issue with U2 and U3 footprints and began layout of PCB tracings
Parts:
- added C1, C3, C7: 0.1u, Package_SO:SOIC-8_3.9x4.9mm_P1.27mm, symbol Device:C
- added C2, C4, C6: 0.1uF, Package_SO:SOIC-8_3.9x4.9mm_P1.27mm, symbol Device:C
- added C5: 1uF, Package_SO:SOIC-8_3.9x4.9mm_P1.27mm, symbol Device:C
- added J1, J2: Conn_01x02_Pin, Package_DIP:DIP-20_W7.62mm, symbol Connector:Conn_01x02_Pin
- added U1: NAU7802KGI, NAU7802KGI:DIP792W45P254L1904H533Q16, symbol NAU7802KGI:NAU7802KGI
- added U2, U3: ACS772LCB-050B-PFF-T, linear_actuator_footprints:XDCR_ACS772LCB-050B-PFF-T, symbol 2026-10-17_14-50-00:ACS772LCB-050B-PFF-T
- added U4: (no value), linear_actuator_footprints:DFR1193, symbol dfr1193:DFR1193
Connections:
- new net: U1.13 (SCLK), U4.3 (SCL_IN)
- new net: U1.14 (SDIO), U4.4 (SDA_IN)
- new net: J1.1 (Pin_1), U2.4
- new net: J1.2 (Pin_2), U2.5
- new net: J2.1 (Pin_1), U3.4
- new net: J2.2 (Pin_2), U3.5
- new net: C3.1, C5.2, U1.16 (AVDD/LDO)
- new net: C7.1, U1.6 (VBG)
- new net +5V: C1.1, C2.1, C4.1, C6.1, U1.1 (REFP), U1.15 (DVDD), U2.1, U3.1, U4.1 (VCC1), U4.9 (VCC2)
- new net GND: C1.2, C2.2, C3.2, C4.2, C5.1, C6.2, C7.2, U1.2 (VIN1N), U1.4 (VIN2N), U1.7 (REFN), U1.8 (AVSS), U1.9 (DVSS), U2.2, U3.2, U4.2 (GND1), U4.8 (GND2)
- new net I_sense_1: U1.3 (VIN1P), U2.3
- new net I_sense_2: U1.5 (VIN2P), U3.3
- no-connect marks 0 -> 6
Other:
- note added: "Pin 5, 6, 7 connected to internal components"

Commit message: Added breakers, updated footprints
Parts:
- removed J1, J2: Conn_01x02_Pin, Package_DIP:DIP-20_W7.62mm, symbol Connector:Conn_01x02_Pin
- added F1, F2: 3557-2, linear_actuator_footprints:FUSE_3557-2, symbol Lin_act_symbols:3557-2
- added J1, J2: Conn_01x04_Socket, linear_actuator_footprints:CONN2_2604-1102_WAG, symbol Connector:Conn_01x04_Socket
- C1, C2, C3, C4, C5, C6, C7: footprint Package_SO:SOIC-8_3.9x4.9mm_P1.27mm -> Capacitor_SMD:C_1206_3216Metric
Connections:
- net at U2.4: now also F2.1_1, F2.1_2
- net at U2.5: now also J1.1 (Pin_1), J1.2 (Pin_2)
- net at U3.4: now also F1.1_1, F1.1_2
- net at U3.5: now also J2.1 (Pin_1), J2.2 (Pin_2)
- new net: F2.2_1, F2.2_2, J1.3 (Pin_3), J1.4 (Pin_4)
- new net: F1.2_1, F1.2_2, J2.3 (Pin_3), J2.4 (Pin_4)
Other:
- moved on the sheet: C4, C6, U2, U3
